Commit message: recommit

File: python/right_hand_mesh/right_hand.urdf (robot description, URDF)
Before this commit: robot for_urdf_export, 16 links, 15 joints
Joints:
- joint index_dip_Revolute-4: axis 1.0 3.9443045261050586e-31 -5.970058958597666e-16 -> 0.9999999999999962 -4.662936703425647e-15 2.521624556202696e-15; origin xyz=9.999999999999788e-05 -0.03610000000000001 -2.886579864025407e-17 rpy=6.736023683033884e-16 -0.0 0.0 -> xyz=0.014450000000000003 -0.03610000000000001 -2.886579864025407e-17 rpy=7.635123965975653e-16 2.8730071914463814e-16 2.335717952496475e-31
- joint index_fingertip_Rigid_index: origin xyz=0.014499999999999994 -0.049499999999999995 -0.009098110000000006 rpy=-3.141592653589793 1.97215226305253e-31 -1.9721522630525293e-31 -> xyz=-2.3092638912203257e-16 -0.04950000000000003 -0.0005000000000000049 rpy=-1.5707963267948966 -1.5707963267948941 0
- joint middle_dip_Revolute-9: axis 1.0 5.497760582556778e-47 -5.970058958597674e-16 -> -0.9999999999999968 1.3322676295501987e-15 -2.2230562504849705e-16; origin xyz=0.00010000000000000009 -0.03610000000000001 -2.886579864025407e-17 rpy=6.736023683033881e-16 3.944304526105061e-31 -1.9721522630525262e-31 -> xyz=0.01445 -0.03610000000000001 -2.886579864025407e-17 rpy=-3.1415926535897927 -5.970058958597673e-16 -1.0770038057096886e-30
- joint middle_fingertip_Rigid_middle: origin xyz=0.014499999999999996 -0.049499999999999995 -0.009098110000000006 rpy=-3.141592653589793 -2.74888029127839e-47 1.9721522630525295e-31 -> xyz=6.661338147750939e-17 0.049499999999999926 0.0005000000000000072 rpy=-3.141592653589793 -5.970058958597633e-16 -7.411401895093593e-31
- joint thumb_dip_Revolute-14: axis 0.0 -1.94289029309401e-16 1.0 -> 3.27515792264423e-15 -1.94289029309406e-16 1.0000000000000018; origin xyz=0.0466 0.0 0.00020000000000000017 rpy=-1.94289029309401e-16 -0.0 -2.097380244072424e-31 -> xyz=0.0466 0.0 -0.014299999999999997 rpy=-1.9428902930940565e-16 -3.2751579226442197e-15 1.189074479488685e-31
- joint thumb_fingertip_Rigid_thumb: origin xyz=0.062099999999999954 -0.009098109999999994 -0.0143 rpy=1.94289029309401e-16 1.2446602076121817e-46 -6.406229996805881e-31 -> xyz=0.062099999999999794 -0.0004999999999999894 4.9999999999794655e-05 rpy=-3.141592653589793 3.2751579226442236e-15 -1.0811969824151546e-30

Commit message: combined fk and ik

File: python/right_hand_mesh/right_hand.urdf (robot description, URDF)
Before this commit: robot for_urdf_export, 16 links, 15 joints
Links:
- removed link index_dip
- removed link index_fingertip
- removed link index_pip
- removed link middle_dip
- removed link middle_fingertip
- removed link middle_pip
- removed link thumb_dip
- removed link thumb_fingertip
- removed link thumb_pip1
- removed link thumb_pip2
- added link index_distal, mass 0.11971825858324693; collision mesh filename=meshes/index_distal.stl scale=0.001 0.001 0.001; visual mesh filename=meshes/index_distal.stl scale=0.001 0.001 0.001
- added link index_inter, mass 0.17326501033259323; collision mesh filename=meshes/index_inter.stl scale=0.001 0.001 0.001; visual mesh filename=meshes/index_inter.stl scale=0.001 0.001 0.001
- added link index_proximal, mass 0.1368678994313018; collision mesh filename=meshes/index_proximal.stl scale=0.001 0.001 0.001; visual mesh filename=meshes/index_proximal.stl scale=0.001 0.001 0.001
- added link middle_distal, mass 0.11971825858324643; collision mesh filename=meshes/middle_distal.stl scale=0.001 0.001 0.001; visual mesh filename=meshes/middle_distal.stl scale=0.001 0.001 0.001
- added link middle_inter, mass 0.17326501033259323; collision mesh filename=meshes/middle_inter.stl scale=0.001 0.001 0.001; visual mesh filename=meshes/middle_inter.stl scale=0.001 0.001 0.001
- added link middle_proximal, mass 0.1368678994313018; collision mesh filename=meshes/middle_proximal.stl scale=0.001 0.001 0.001; visual mesh filename=meshes/middle_proximal.stl scale=0.001 0.001 0.001
- added link thumb_distal, mass 0.25656730685939594; collision mesh filename=meshes/thumb_distal.stl scale=0.001 0.001 0.001; visual mesh filename=meshes/thumb_distal.stl scale=0.001 0.001 0.001
- added link thumb_mcp1, mass 0.1368678994313018; collision mesh filename=meshes/thumb_mcp1.stl scale=0.001 0.001 0.001; visual mesh filename=meshes/thumb_mcp1.stl scale=0.001 0.001 0.001
- added link thumb_mcp2, mass 0.01935609811919093; collision mesh filename=meshes/thumb_mcp2.stl scale=0.001 0.001 0.001; visual mesh filename=meshes/thumb_mcp2.stl scale=0.001 0.001 0.001
- added link thumb_proximal, mass 0.17555980876954594; collision mesh filename=meshes/thumb_proximal.stl scale=0.001 0.001 0.001; visual mesh filename=meshes/thumb_proximal.stl scale=0.001 0.001 0.001
Joints:
- removed joint index_dip_Revolute-4
- removed joint index_fingertip_Rigid_index
- removed joint index_mcp_joint_Revolute-2
- removed joint index_pip_Revolute-3
- removed joint middle_dip_Revolute-9
- removed joint middle_fingertip_Rigid_middle
- removed joint middle_mcp_joint_Revolute-7
- removed joint middle_pip_Revolute-8
- removed joint thumb_dip_Revolute-14
- removed joint thumb_fingertip_Rigid_thumb
- removed joint thumb_pip1_Revolute-12
- removed joint thumb_pip2_Revolute-13
- added joint index_distal_Rigid_index: type fixed, parent index_distal, child index_realtip, origin xyz=-2.3092638912203257e-16 -0.04950000000000003 -0.0005000000000000049 rpy=4.947476175360935e-17 -2.8730071914463834e-16 -1.8006098300157965e-31
- added joint index_inter_Revolute-9: type continuous, parent index_inter, child index_distal, origin xyz=0.014450000000000003 -0.03610000000000001 -2.886579864025407e-17 rpy=7.635123965975653e-16 2.8730071914463814e-16 2.335717952496475e-31, axis 0.9999999999999962 -4.662936703425647e-15 2.521624556202696e-15
- added joint index_mcp_joint_Revolute-7: type continuous, parent index_mcp_joint, child index_proximal, origin xyz=0.012199999999999973 0.03810000000000001 0.014499999999999985 rpy=3.1415926535897913 3.944304526105059e-31 2.8022431570960223e-32, axis 1.0 1.0970034457409265e-32 -5.997407798921492e-16
- added joint index_proximal_Revolute-8: type continuous, parent index_proximal, child index_inter, origin xyz=-0.012999999999999987 -0.015000000000000027 0.014399999999999977 rpy=-8.129871583511721e-16 1.570796326794895 0, axis 1.0 3.944304526105059e-31 1.21876284056415e-17
- added joint middle_distal_Rigid_middle: type fixed, parent middle_distal, child middle_realtip, origin xyz=6.661338147750939e-17 -0.049499999999999926 -0.0005000000000000027 rpy=4.94747617536117e-17 -2.8730071914463617e-16 7.4274998325118455e-31
- added joint middle_inter_Revolute-14: type continuous, parent middle_inter, child middle_distal, origin xyz=0.01445 -0.03610000000000001 -2.886579864025407e-17 rpy=7.63512396597558e-16 2.873007191446387e-16 -5.552891099713655e-31, axis 0.9999999999999968 1.3322676295501985e-15 6.620009899558993e-16
- added joint middle_mcp_joint_Revolute-12: type continuous, parent middle_mcp_joint, child middle_proximal, origin xyz=0.01219999999999999 0.03810000000000001 0.014499999999999985 rpy=3.1415926535897913 2.5353555998624977e-47 6.457697323376579e-32, axis 1.0 -3.164352580666406e-32 -5.9974077989215e-16
- added joint middle_proximal_Revolute-13: type continuous, parent middle_proximal, child middle_inter, origin xyz=-0.012999999999999989 -0.015000000000000027 0.014399999999999977 rpy=-8.129871583511721e-16 1.570796326794895 0, axis 1.0 0.0 1.21876284056415e-17
- added joint thumb_distal_Rigid_thumb: type fixed, parent thumb_distal, child thumb_realtip, origin xyz=0.062099999999999794 -0.0004999999999999894 4.9999999999794655e-05 rpy=-3.141592653589793 3.2751579226442236e-15 -1.0811969824151546e-30
- added joint thumb_mcp1_Revolute-2: type continuous, parent thumb_mcp1, child thumb_mcp2, origin xyz=0.01429999999999997 3.1086244689504386e-17 -0.012999999999999998 rpy=1.5707963267948981 3.944304526105086e-31 -1.2030572237243167e-30, axis -1.0 1.2818309776324673e-45 -3.178737046341918e-17
- added joint thumb_mcp2_Revolute-3: type continuous, parent thumb_mcp2, child thumb_proximal, origin xyz=0.01700000000000001 1.7763568394002505e-17 -0.014499999999999996 rpy=-3.1415926535897922 1.2030572237243175e-30 -6.767517584326818e-32, axis 0.0 0.0 1.0
- added joint thumb_proximal_Revolute-4: type continuous, parent thumb_proximal, child thumb_distal, origin xyz=0.0466 0.0 -0.014299999999999997 rpy=-1.9428902930940565e-16 -3.2751579226442197e-15 1.189074479488685e-31, axis 3.27515792264423e-15 -1.94289029309406e-16 1.0000000000000018
- joint palm_Revolute-1: axis 0.0 3.3709870223533754e-16 1.0 -> 0.0 -2.2920118444087085e-15 1.0; child index_mcp_joint -> thumb_mcp1; origin xyz=0.0637 -0.013000000000000001 0.017275000000000002 rpy=-3.141592653589793 -1.5707963267948966 0 -> xyz=0.06849999999999999 0.0495 0.0131 rpy=1.5707963267948943 -0.0 0.0
- joint palm_Revolute-11: axis 0.0 -2.2920118444087085e-15 1.0 -> 0.0 3.9260985346659443e-16 1.0; child thumb_pip1 -> middle_mcp_joint; origin xyz=0.06849999999999999 0.0495 0.0131 rpy=1.5707963267948943 -0.0 0.0 -> xyz=0.005699999999999999 -0.013000000000000001 0.017275000000000002 rpy=-3.1415926535897927 -1.5707963267948966 0
- joint palm_Revolute-6: axis 0.0 3.9260985346659443e-16 1.0 -> 0.0 3.3709870223533754e-16 1.0; child middle_mcp_joint -> index_mcp_joint; origin xyz=0.005699999999999999 -0.013000000000000001 0.017275000000000002 rpy=-3.1415926535897927 -1.5707963267948966 0 -> xyz=0.0637 -0.013000000000000001 0.017275000000000002 rpy=-3.141592653589793 -1.5707963267948966 0
