Commit message: it's a wrap

File: python/left_hand_mesh/left_hand.urdf (robot description, URDF)
Before this commit: robot for_urdf_left, 16 links, 15 joints
Joints:
- joint index_mcp_joint_Revolute-7: axis -1.0 1.0615834244799634e-32 -5.9974077989215e-16 -> 1.0 1.0615834244799634e-32 -5.9974077989215e-16
- joint middle_mcp_joint_Revolute-12: axis -1.0 -5.095803370108072e-33 -5.9974077989215e-16 -> 1.0 -5.095803370108072e-33 -5.9974077989215e-16
- joint palm_Revolute-1: axis 0.0 -2.2920118444087085e-15 1.0 -> 0.0 -2.2920118444087085e-15 -1.0
- joint thumb_proximal_Revolute-4: axis -3.27515792264423e-15 1.9428902930940634e-16 -1.0000000000000018 -> -3.27515792264423e-15 1.9428902930940634e-16 1.0000000000000018

File: python/right_hand_mesh/right_hand.urdf (robot description, URDF)
Before this commit: robot for_urdf_right, 16 links, 15 joints
Joints:
- joint index_mcp_joint_Revolute-7: axis 1.0 1.0970034457409265e-32 -5.997407798921492e-16 -> -1.0 1.0970034457409265e-32 -5.997407798921492e-16
- joint middle_mcp_joint_Revolute-12: axis 1.0 -3.164352580666406e-32 -5.9974077989215e-16 -> -1.0 -3.164352580666406e-32 -5.9974077989215e-16
- joint palm_Revolute-1: axis 0.0 -2.2920118444087085e-15 1.0 -> 0.0 -2.2920118444087085e-15 -1.0
- joint thumb_mcp1_Revolute-2: axis -1.0 1.2818309776324673e-45 -3.178737046341918e-17 -> 1.0 1.2818309776324673e-45 -3.178737046341918e-17
- joint thumb_mcp2_Revolute-3: axis 0.0 0.0 1.0 -> 0.0 0.0 -1.0
- joint thumb_proximal_Revolute-4: axis 3.27515792264423e-15 -1.94289029309406e-16 1.0000000000000018 -> 3.27515792264423e-15 -1.94289029309406e-16 -1.0000000000000018
